Commit message: ContinuO finaly walks in simgit add -ugit add -ugit add -ugit add -ugit add -ugit add -ugit add -ugit add -ugit add -ugit add -u

File: florant/f_quadruped_control/urdf/ContinuO_lidar.xacro (robot description, xacro)
@@ -1,10 +1,19 @@
 <?xml version="1.0" encoding="utf-8"?>
 <robot xmlns:xacro="http://ros.org/wiki/xacro" name="ContinuO">
+  <!-- To make the robot fly -->
+  <!-- Wingardium leviossssssssssssssssssa -->
+  <!-- <link name="world" /> -->
+  <!---->
+  <!-- <joint name="fixed_to_world" type="fixed"> -->
+  <!--   <parent link="world" /> -->
+  <!--   <child link="base_link" /> -->
+  <!--   <origin xyz="0 0 0.5" rpy="0 0 0" /> -->
+  <!-- </joint> -->
   <!-- INCLUSIONS -->
-  <xacro:include filename="$(find f_quadruped_control)/urdf/materials.xacro"/>
-  <xacro:include filename="$(find f_quadruped_control)/urdf/sensors.xacro"/>
-  <xacro:include filename="$(find f_quadruped_control)/urdf/legs.xacro"/>
-  <xacro:include filename="$(find f_quadruped_control)/urdf/transmissions.xacro"/>
-  <xacro:include filename="$(find f_quadruped_control)/urdf/gazebo.xacro"/>
+  <xacro:include filename="$(find f_quadruped_control)/urdf/materials.xacro" />
+  <xacro:include filename="$(find f_quadruped_control)/urdf/sensors.xacro" />
+  <xacro:include filename="$(find f_quadruped_control)/urdf/legs.xacro" />
+  <xacro:include filename="$(find f_quadruped_control)/urdf/transmissions.xacro" />
+  <xacro:include filename="$(find f_quadruped_control)/urdf/gazebo.xacro" />
   <!-- LIEN DE BASE -->
   <link name="base_link" />
@@ -18,5 +27,5 @@
       <mass value="15.342" />
       <inertia ixx="0.131477" ixy="-0.000035" ixz="0.000257"
-               iyy="0.328587" iyz="0.000031" izz="0.423802" />
+        iyy="0.328587" iyz="0.000031" izz="0.423802" />
     </inertial>
     <visual>
@@ -25,5 +34,5 @@
         <mesh filename="package://f_quadruped_control/meshes/base.dae" />
       </geometry>
-      <material name="red"/>
+      <material name="red" />
     </visual>
     <collision>

File: florant/f_quadruped_control/urdf/gazebo.xacro (robot description, xacro)
@@ -5,4 +5,5 @@
     <plugin name="gazebo_ros_control" filename="libgazebo_ros_control.so">
       <robotNamespace>/</robotNamespace>
+      <controlPeriod>0.004</controlPeriod> <!-- the controller reads my commands at 250Hz -->
     </plugin>
   </gazebo>
@@ -68,10 +69,10 @@
     <sensor name="imu_sensor" type="imu">
       <always_on>true</always_on>
-      <update_rate>200</update_rate>
+      <update_rate>100</update_rate>
       <visualize>false</visualize>
       <plugin filename="libgazebo_ros_imu_sensor.so" name="imu_plugin">
         <topicName>/imu</topicName>
         <bodyName>imu_link</bodyName>
-        <updateRateHZ>200.0</updateRateHZ>
+        <updateRateHZ>100.0</updateRateHZ>
         <gaussianNoise>0.0</gaussianNoise>
         <xyzOffset>0 0 0</xyzOffset>
@@ -93,8 +94,8 @@
     </gazebo>
   </xacro:macro>
-  <xacro:foot_friction link_name="FL_FOOT"/>
-  <xacro:foot_friction link_name="FR_FOOT"/>
-  <xacro:foot_friction link_name="HL_FOOT"/>
-  <xacro:foot_friction link_name="HR_FOOT"/>
+  <xacro:foot_friction link_name="FL_FOOT" />
+  <xacro:foot_friction link_name="FR_FOOT" />
+  <xacro:foot_friction link_name="HL_FOOT" />
+  <xacro:foot_friction link_name="HR_FOOT" />
   <gazebo reference="base">
     <kp>2e5</kp>

File: florant/f_quadruped_control/urdf/legs.xacro (robot description, xacro)
@@ -6,14 +6,19 @@
       <origin xyz="0.051772 0.021258 -0.000161" rpy="0 0 0" />
       <mass value="1.276" />
-      <inertia ixx="0.001862" ixy="0.000034" ixz="0.000001" iyy="0.001745" iyz="0.000000" izz="0.001887" />
-    </inertial>
-    <visual>
-      <origin xyz="0 0 0" rpy="0 0 0" />
-      <geometry><mesh filename="package://quadruped_description/meshes/FL_SHOULDER.dae" /></geometry>
-      <material name="black"/>
+      <inertia ixx="0.001862" ixy="0.000034" ixz="0.000001" iyy="0.001745" iyz="0.000000"
+        izz="0.001887" />
+    </inertial>
+    <visual>
+      <origin xyz="0 0 0" rpy="0 0 0" />
+      <geometry>
+        <mesh filename="package://quadruped_description/meshes/FL_SHOULDER.dae" />
+      </geometry>
+      <material name="black" />
     </visual>
     <collision>
       <origin xyz="0.054 0 0" rpy="0 0 0" />
-      <geometry><box size="0.1 0.1 0.1" /></geometry>
+      <geometry>
+        <box size="0.1 0.1 0.1" />
+      </geometry>
     </collision>
   </link>
@@ -24,5 +29,5 @@
     <axis xyz="1 0 0" />
     <dynamics damping="0.7" friction="0.0" />
-    <limit lower="-3.14" upper="3.14" effort="85.0" velocity="16.75" />
+    <limit lower="-3.14" upper="3.14" effort="125.0" velocity="16.75" />
   </joint>
   <link name="FL_UPPER_LEG">
@@ -30,14 +35,19 @@
       <origin xyz="0.000009 0.025634 -0.165001" rpy="0 0 0" />
       <mass value="1.367" />
-      <inertia ixx="0.016273" ixy="-0.000000" ixz="0.000012" iyy="0.016691" iyz="0.000130" izz="0.001167" />
-    </inertial>
-    <visual>
-      <origin xyz="0 0 0" rpy="0 0 0" />
-      <geometry><mesh filename="package://quadruped_description/meshes/FL_UPPER_LEG.dae" /></geometry>
-      <material name="black2"/>
+      <inertia ixx="0.016273" ixy="-0.000000" ixz="0.000012" iyy="0.016691" iyz="0.000130"
+        izz="0.001167" />
+    </inertial>
+    <visual>
+      <origin xyz="0 0 0" rpy="0 0 0" />
+      <geometry>
+        <mesh filename="package://quadruped_description/meshes/FL_UPPER_LEG.dae" />
+      </geometry>
+      <material name="black2" />
     </visual>
     <collision>
       <origin xyz="0 0.032 -0.1232" rpy="0 0 0" />
-      <geometry><box size="0.1 0.05 0.3" /></geometry>
+      <geometry>
+        <box size="0.1 0.05 0.3" />
+      </geometry>
     </collision>
   </link>
@@ -48,5 +58,5 @@
     <axis xyz="0 1 0" />
     <dynamics damping="0.9" friction="0.0" />
-    <limit lower="-3.14" upper="3.14" effort="80.0" velocity="23.04" />
+    <limit lower="-3.14" upper="3.14" effort="120.0" velocity="23.04" />
   </joint>
   <link name="FL_LOWER_LEG">
@@ -54,14 +64,19 @@
       <origin xyz="-0.041308 0.034919 -0.047598" rpy="0 0 0" />
       <mass value="0.759" />
-      <inertia ixx="0.007966" ixy="-0.000009" ixz="0.001312" iyy="0.009247" iyz="-0.000002" izz="0.001638" />
-    </inertial>
-    <visual>
-      <origin xyz="0 0 0" rpy="0 0 0" />
-      <geometry><mesh filename="package://quadruped_description/meshes/FL_LOWER_LEG.dae" /></geometry>
-      <material name="black3"/>
+      <inertia ixx="0.007966" ixy="-0.000009" ixz="0.001312" iyy="0.009247" iyz="-0.000002"
+        izz="0.001638" />
+    </inertial>
+    <visual>
+      <origin xyz="0 0 0" rpy="0 0 0" />
+      <geometry>
+        <mesh filename="package://quadruped_description/meshes/FL_LOWER_LEG.dae" />
+      </geometry>
+      <material name="black3" />
     </visual>
     <collision>
       <origin xyz="-0.0772 0.035 -0.09" rpy="0 0 0" />
-      <geometry><cylinder length="0.3" radius="0.02"/></geometry>
+      <geometry>
+        <cylinder length="0.3" radius="0.02" />
+      </geometry>
     </collision>
   </link>
@@ -72,5 +87,5 @@
     <axis xyz="0 1 0" />
     <dynamics damping="0.9" friction="0.0" />
-    <limit lower="-3.14" upper="3.14" effort="80.0" velocity="23.04" />
+    <limit lower="-3.14" upper="3.14" effort="120.0" velocity="23.04" />
   </joint>
   <link name="FL_FOOT">
@@ -78,14 +93,19 @@
       <origin xyz="0.035896 -0.000081 0.186367" rpy="0 0 0" />
       <mass value="0.01" />
-      <inertia ixx="0.007966" ixy="-0.000009" ixz="0.001312" iyy="0.009247" iyz="-0.000002" izz="0.001638" />
-    </inertial>
-    <visual>
-      <origin xyz="0 0 0" rpy="0 0 0" />
-      <geometry><mesh filename="package://quadruped_description/meshes/FL_FOOT.dae" /></geometry>
-      <material name="red"/>
+      <inertia ixx="0.007966" ixy="-0.000009" ixz="0.001312" iyy="0.009247" iyz="-0.000002"
+        izz="0.001638" />
+    </inertial>
+    <visual>
+      <origin xyz="0 0 0" rpy="0 0 0" />
+      <geometry>
+        <mesh filename="package://quadruped_description/meshes/FL_FOOT.dae" />
+      </geometry>
+      <material name="red" />
     </visual>
     <collision>
       <origin xyz="0 0 -0.02" rpy="0 0 0" />
-      <geometry><sphere radius="0.0267" /></geometry>
+      <geometry>
+        <sphere radius="0.0267" />
+      </geometry>
     </collision>
   </link>
@@ -100,14 +120,19 @@
       <origin xyz="0.051772 -0.021258 -0.000161" rpy="0 0 0" />
       <mass value="1.276" />
-      <inertia ixx="0.001862" ixy="-0.000034" ixz="0.000001" iyy="0.001745" iyz="-0.000000" izz="0.001887" />
-    </inertial>
-    <visual>
-      <origin xyz="0 0 0" rpy="0 0 0" />
-      <geometry><mesh filename="package://quadruped_description/meshes/FR_SHOULDER.dae" /></geometry>
-      <material name="black"/>
+      <inertia ixx="0.001862" ixy="-0.000034" ixz="0.000001" iyy="0.001745" iyz="-0.000000"
+        izz="0.001887" />
+    </inertial>
+    <visual>
+      <origin xyz="0 0 0" rpy="0 0 0" />
+      <geometry>
+        <mesh filename="package://quadruped_description/meshes/FR_SHOULDER.dae" />
+      </geometry>
+      <material name="black" />
     </visual>
     <collision>
       <origin xyz="0.054 0 0" rpy="0 0 0" />
-      <geometry><box size="0.1 0.1 0.1" /></geometry>
+      <geometry>
+        <box size="0.1 0.1 0.1" />
+      </geometry>
     </collision>
   </link>
@@ -118,5 +143,5 @@
     <axis xyz="1 0 0" />
     <dynamics damping="0.7" friction="0.0" />
-    <limit lower="-3.14" upper="3.14" effort="85.0" velocity="16.75" />
+    <limit lower="-3.14" upper="3.14" effort="125.0" velocity="16.75" />
   </joint>
   <link name="FR_UPPER_LEG">
@@ -124,14 +149,19 @@
       <origin xyz="0.000009 -0.025634 -0.165001" rpy="0 0 0" />
       <mass value="1.367" />
-      <inertia ixx="0.016273" ixy="0.000000" ixz="0.000012" iyy="0.016691" iyz="-0.000130" izz="0.001167" />
-    </inertial>
-    <visual>
-      <origin xyz="0 0 0" rpy="0 0 0" />
-      <geometry><mesh filename="package://quadruped_description/meshes/FR_UPPER_LEG.dae" /></geometry>
-      <material name="black2"/>
+      <inertia ixx="0.016273" ixy="0.000000" ixz="0.000012" iyy="0.016691" iyz="-0.000130"
+        izz="0.001167" />
+    </inertial>
+    <visual>
+      <origin xyz="0 0 0" rpy="0 0 0" />
+      <geometry>
+        <mesh filename="package://quadruped_description/meshes/FR_UPPER_LEG.dae" />
+      </geometry>
+      <material name="black2" />
     </visual>
     <collision>
       <origin xyz="0 -0.028 -0.1232" rpy="0 0 0" />
-      <geometry><box size="0.1 0.05 0.3" /></geometry>
+      <geometry>
+        <box size="0.1 0.05 0.3" />
+      </geometry>
     </collision>
   </link>
@@ -142,5 +172,5 @@
     <axis xyz="0 1 0" />
     <dynamics damping="0.9" friction="0.0" />
-    <limit lower="-3.14" upper="3.14" effort="80.0" velocity="23.04" />
+    <limit lower="-3.14" upper="3.14" effort="120.0" velocity="23.04" />
   </joint>
   <link name="FR_LOWER_LEG">
@@ -148,14 +178,19 @@
       <origin xyz="-0.041308 -0.034919 -0.047598" rpy="0 0 0" />
       <mass value="0.759" />
-      <inertia ixx="0.007966" ixy="0.000009" ixz="0.001312" iyy="0.009247" iyz="0.000002" izz="0.001638" />
-    </inertial>
-    <visual>
-      <origin xyz="0 0 0" rpy="0 0 0" />
-      <geometry><mesh filename="package://quadruped_description/meshes/FR_LOWER_LEG.dae" /></geometry>
-      <material name="black3"/>
+      <inertia ixx="0.007966" ixy="0.000009" ixz="0.001312" iyy="0.009247" iyz="0.000002"
+        izz="0.001638" />
+    </inertial>
+    <visual>
+      <origin xyz="0 0 0" rpy="0 0 0" />
+      <geometry>
+        <mesh filename="package://quadruped_description/meshes/FR_LOWER_LEG.dae" />
+      </geometry>
+      <material name="black3" />
     </visual>
     <collision>
       <origin xyz="-0.0772 -0.035 -0.09" rpy="0 0 0" />
-      <geometry><cylinder length="0.3" radius="0.02"/></geometry>
+      <geometry>
+        <cylinder length="0.3" radius="0.02" />
+      </geometry>
     </collision>
   </link>
@@ -166,5 +201,5 @@
     <axis xyz="0 1 0" />
     <dynamics damping="0.9" friction="0.0" />
-    <limit lower="-3.14" upper="3.14" effort="80.0" velocity="23.04" />
+    <limit lower="-3.14" upper="3.14" effort="120.0" velocity="23.04" />
   </joint>
   <link name="FR_FOOT">
@@ -172,14 +207,19 @@
       <origin xyz="0.035896 0.000081 0.186367" rpy="0 0 0" />
       <mass value="0.01" />
-      <inertia ixx="0.007966" ixy="0.000009" ixz="0.001312" iyy="0.009247" iyz="0.000002" izz="0.001638" />
-    </inertial>
-    <visual>
-      <origin xyz="0 0 0" rpy="0 0 0" />
-      <geometry><mesh filename="package://quadruped_description/meshes/FR_FOOT.dae" /></geometry>
-      <material name="red"/>
+      <inertia ixx="0.007966" ixy="0.000009" ixz="0.001312" iyy="0.009247" iyz="0.000002"
+        izz="0.001638" />
+    </inertial>
+    <visual>
+      <origin xyz="0 0 0" rpy="0 0 0" />
+      <geometry>
+        <mesh filename="package://quadruped_description/meshes/FR_FOOT.dae" />
+      </geometry>
+      <material name="red" />
     </visual>
     <collision>
       <origin xyz="0 0 -0.02" rpy="0 0 0" />
-      <geometry><sphere radius="0.0267" /></geometry>
+      <geometry>
+        <sphere radius="0.0267" />
+      </geometry>
     </collision>
   </link>
@@ -194,14 +234,19 @@
       <origin xyz="-0.051779 0.021258 0.000042" rpy="0 0 0" />
       <mass value="1.276" />
-      <inertia ixx="0.001862" ixy="-0.000034" ixz="-0.000000" iyy="0.001745" iyz="-0.000000" izz="0.001886" />
-    </inertial>
-    <visual>
-      <origin xyz="0 0 0" rpy="0 0 0" />
-      <geometry><mesh filename="package://quadruped_description/meshes/HL_SHOULDER.dae" /></geometry>
-      <material name="black"/>
+      <inertia ixx="0.001862" ixy="-0.000034" ixz="-0.000000" iyy="0.001745" iyz="-0.000000"
+        izz="0.001886" />
+    </inertial>
+    <visual>
+      <origin xyz="0 0 0" rpy="0 0 0" />
+      <geometry>
+        <mesh filename="package://quadruped_description/meshes/HL_SHOULDER.dae" />
+      </geometry>
+      <material name="black" />
     </visual>
     <collision>
       <origin xyz="-0.054 0 0" rpy="0 0 0" />
-      <geometry><box size="0.1 0.1 0.1" /></geometry>
+      <geometry>
+        <box size="0.1 0.1 0.1" />
+      </geometry>
     </collision>
   </link>
@@ -212,5 +257,5 @@
     <axis xyz="1 0 0" />
     <dynamics damping="0.7" friction="0.0" />
-    <limit lower="-3.14" upper="3.14" effort="85.0" velocity="16.75" />
+    <limit lower="-3.14" upper="3.14" effort="125.0" velocity="16.75" />
   </joint>
   <link name="HL_UPPER_LEG">
@@ -218,14 +263,19 @@
       <origin xyz="0.000003 0.025470 -0.134787" rpy="0 0 0" />
       <mass value="1.315" />
-      <inertia ixx="0.011053" ixy="-0.000000" ixz="0.000013" iyy="0.011463" iyz="0.000105" izz="0.001146" />
-    </inertial>
-    <visual>
-      <origin xyz="0 0 0" rpy="0 0 0" />
-      <geometry><mesh filename="package://quadruped_description/meshes/HL_UPPER_LEG.dae" /></geometry>
-      <material name="black1"/>
+      <inertia ixx="0.011053" ixy="-0.000000" ixz="0.000013" iyy="0.011463" iyz="0.000105"
+        izz="0.001146" />
+    </inertial>
+    <visual>
+      <origin xyz="0 0 0" rpy="0 0 0" />
+      <geometry>
+        <mesh filename="package://quadruped_description/meshes/HL_UPPER_LEG.dae" />
+      </geometry>
+      <material name="black1" />
     </visual>
     <collision>
       <origin xyz="0 0.028 -0.1005" rpy="0 0 0" />
-      <geometry><box size="0.08 0.05 0.26" /></geometry>
+      <geometry>
+        <box size="0.08 0.05 0.26" />
+      </geometry>
     </collision>
   </link>
@@ -236,5 +286,5 @@
     <axis xyz="0 1 0" />
     <dynamics damping="0.9" friction="0.0" />
-    <limit lower="-3.14" upper="3.14" effort="85.0" velocity="16.75" />
+    <limit lower="-3.14" upper="3.14" effort="125.0" velocity="16.75" />
   </joint>
   <link name="HL_LOWER_LEG">
@@ -242,14 +292,19 @@
       <origin xyz="0.000005 0.041724 -0.160773" rpy="0 0 0" />
       <mass value="1.406" />
-      <inertia ixx="0.017322" ixy="-0.000000" ixz="0.000013" iyy="0.017702" iyz="-0.000074" izz="0.001218" />
-    </inertial>
-    <visual>
-      <origin xyz="0 0 0" rpy="0 0 0" />
-      <geometry><mesh filename="package://quadruped_description/meshes/HL_LOWER_LEG.dae" /></geometry>
-      <material name="black2"/>
+      <inertia ixx="0.017322" ixy="-0.000000" ixz="0.000013" iyy="0.017702" iyz="-0.000074"
+        izz="0.001218" />
+    </inertial>
+    <visual>
+      <origin xyz="0 0 0" rpy="0 0 0" />
+      <geometry>
+        <mesh filename="package://quadruped_description/meshes/HL_LOWER_LEG.dae" />
+      </geometry>
+      <material name="black2" />
     </visual>
     <collision>
       <origin xyz="0 0.045 -0.1233" rpy="0 0 0" />
-      <geometry><box size="0.06 0.05 0.35" /></geometry>
+      <geometry>
+        <box size="0.06 0.05 0.35" />
+      </geometry>
     </collision>
   </link>
@@ -260,5 +315,5 @@
     <axis xyz="0 1 0" />
     <dynamics damping="0.9" friction="0.0" />
-    <limit lower="-3.14" upper="3.14" effort="80.0" velocity="23.04" />
+    <limit lower="-3.14" upper="3.14" effort="120.0" velocity="23.04" />
   </joint>
   <link name="HL_SHANK">
@@ -266,14 +321,19 @@
       <origin xyz="-0.040122 0.034916 -0.027409" rpy="0 0 0" />
       <mass value="0.734" />
-      <inertia ixx="0.003597" ixy="-0.000009" ixz="0.000762" iyy="0.004846" iyz="-0.000001" izz="0.001602" />
-    </inertial>
-    <visual>
-      <origin xyz="0 0 0" rpy="0 0 0" />
-      <geometry><mesh filename="package://quadruped_description/meshes/HL_SHANK.dae" /></geometry>
-      <material name="black3"/>
+      <inertia ixx="0.003597" ixy="-0.000009" ixz="0.000762" iyy="0.004846" iyz="-0.000001"
+        izz="0.001602" />
+    </inertial>
+    <visual>
+      <origin xyz="0 0 0" rpy="0 0 0" />
+      <geometry>
+        <mesh filename="package://quadruped_description/meshes/HL_SHANK.dae" />
+      </geometry>
+      <material name="black3" />
     </visual>
     <collision>
       <origin xyz="-0.0772 0.035 -0.045" rpy="0 0 0" />
-      <geometry><cylinder length="0.21" radius="0.02"/></geometry>
+      <geometry>
+        <cylinder length="0.21" radius="0.02" />
+      </geometry>
     </collision>
   </link>
@@ -284,5 +344,5 @@
     <axis xyz="0 1 0" />
     <dynamics damping="0.9" friction="0.0" />
-    <limit lower="-3.14" upper="3.14" effort="80.0" velocity="23.04" />
+    <limit lower="-3.14" upper="3.14" effort="120.0" velocity="23.04" />
   </joint>
   <link name="HL_FOOT">
@@ -290,14 +350,19 @@
       <origin xyz="0.037082 -0.000084 0.116555" rpy="0 0 0" />
       <mass value="0.01" />
-      <inertia ixx="0.003597" ixy="-0.000009" ixz="0.000762" iyy="0.004846" iyz="-0.000001" izz="0.001602" />
-    </inertial>
-    <visual>
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