Commit message: end of day

File: florant/f_quadruped_control/urdf/ContinuO_lidar.xacro (robot description, xacro)
@@ -3,11 +3,10 @@
   <!-- To make the robot fly -->
   <!-- Wingardium leviossssssssssssssssssa -->
-  <!-- <link name="world" /> -->
-  <!---->
-  <!-- <joint name="fixed_to_world" type="fixed"> -->
-  <!--   <parent link="world" /> -->
-  <!--   <child link="base_link" /> -->
-  <!--   <origin xyz="0 0 0.5" rpy="0 0 0" /> -->
-  <!-- </joint> -->
+  <link name="world" />
+  <joint name="fixed_to_world" type="fixed">
+    <parent link="world" />
+    <child link="base_link" />
+    <origin xyz="0 0 0.5" rpy="0 0 0" />
+  </joint>
   <!-- INCLUSIONS -->
   <xacro:include filename="$(find f_quadruped_control)/urdf/materials.xacro" />

File: florant/f_quadruped_control/urdf/legs.xacro (robot description, xacro)
@@ -12,5 +12,5 @@
       <origin xyz="0 0 0" rpy="0 0 0" />
       <geometry>
-        <mesh filename="package://quadruped_description/meshes/FL_SHOULDER.dae" />
+        <mesh filename="package://f_quadruped_control/meshes/FL_SHOULDER.dae" />
       </geometry>
       <material name="black" />
@@ -41,5 +41,5 @@
       <origin xyz="0 0 0" rpy="0 0 0" />
       <geometry>
-        <mesh filename="package://quadruped_description/meshes/FL_UPPER_LEG.dae" />
+        <mesh filename="package://f_quadruped_control/meshes/FL_UPPER_LEG.dae" />
       </geometry>
       <material name="black2" />
@@ -70,5 +70,5 @@
       <origin xyz="0 0 0" rpy="0 0 0" />
       <geometry>
-        <mesh filename="package://quadruped_description/meshes/FL_LOWER_LEG.dae" />
+        <mesh filename="package://f_quadruped_control/meshes/FL_LOWER_LEG.dae" />
       </geometry>
       <material name="black3" />
@@ -99,5 +99,5 @@
       <origin xyz="0 0 0" rpy="0 0 0" />
       <geometry>
-        <mesh filename="package://quadruped_description/meshes/FL_FOOT.dae" />
+        <mesh filename="package://f_quadruped_control/meshes/FL_FOOT.dae" />
       </geometry>
       <material name="red" />
@@ -126,5 +126,5 @@
       <origin xyz="0 0 0" rpy="0 0 0" />
       <geometry>
-        <mesh filename="package://quadruped_description/meshes/FR_SHOULDER.dae" />
+        <mesh filename="package://f_quadruped_control/meshes/FR_SHOULDER.dae" />
       </geometry>
       <material name="black" />
@@ -155,5 +155,5 @@
       <origin xyz="0 0 0" rpy="0 0 0" />
       <geometry>
-        <mesh filename="package://quadruped_description/meshes/FR_UPPER_LEG.dae" />
+        <mesh filename="package://f_quadruped_control/meshes/FR_UPPER_LEG.dae" />
       </geometry>
       <material name="black2" />
@@ -184,5 +184,5 @@
       <origin xyz="0 0 0" rpy="0 0 0" />
       <geometry>
-        <mesh filename="package://quadruped_description/meshes/FR_LOWER_LEG.dae" />
+        <mesh filename="package://f_quadruped_control/meshes/FR_LOWER_LEG.dae" />
       </geometry>
       <material name="black3" />
@@ -213,5 +213,5 @@
       <origin xyz="0 0 0" rpy="0 0 0" />
       <geometry>
-        <mesh filename="package://quadruped_description/meshes/FR_FOOT.dae" />
+        <mesh filename="package://f_quadruped_control/meshes/FR_FOOT.dae" />
       </geometry>
       <material name="red" />
@@ -240,5 +240,5 @@
       <origin xyz="0 0 0" rpy="0 0 0" />
       <geometry>
-        <mesh filename="package://quadruped_description/meshes/HL_SHOULDER.dae" />
+        <mesh filename="package://f_quadruped_control/meshes/HL_SHOULDER.dae" />
       </geometry>
       <material name="black" />
@@ -269,5 +269,5 @@
       <origin xyz="0 0 0" rpy="0 0 0" />
       <geometry>
-        <mesh filename="package://quadruped_description/meshes/HL_UPPER_LEG.dae" />
+        <mesh filename="package://f_quadruped_control/meshes/HL_UPPER_LEG.dae" />
       </geometry>
       <material name="black1" />
@@ -298,5 +298,5 @@
       <origin xyz="0 0 0" rpy="0 0 0" />
       <geometry>
-        <mesh filename="package://quadruped_description/meshes/HL_LOWER_LEG.dae" />
+        <mesh filename="package://f_quadruped_control/meshes/HL_LOWER_LEG.dae" />
       </geometry>
       <material name="black2" />
@@ -327,5 +327,5 @@
       <origin xyz="0 0 0" rpy="0 0 0" />
       <geometry>
-        <mesh filename="package://quadruped_description/meshes/HL_SHANK.dae" />
+        <mesh filename="package://f_quadruped_control/meshes/HL_SHANK.dae" />
       </geometry>
       <material name="black3" />
@@ -356,5 +356,5 @@
       <origin xyz="0 0 0" rpy="0 0 0" />
       <geometry>
-        <mesh filename="package://quadruped_description/meshes/HL_FOOT.dae" />
+        <mesh filename="package://f_quadruped_control/meshes/HL_FOOT.dae" />
       </geometry>
       <material name="red" />
@@ -383,5 +383,5 @@
       <origin xyz="0 0 0" rpy="0 0 0" />
       <geometry>
-        <mesh filename="package://quadruped_description/meshes/HR_SHOULDER.dae" />
+        <mesh filename="package://f_quadruped_control/meshes/HR_SHOULDER.dae" />
       </geometry>
       <material name="black" />
@@ -412,5 +412,5 @@
       <origin xyz="0 0 0" rpy="0 0 0" />
       <geometry>
-        <mesh filename="package://quadruped_description/meshes/HR_UPPER_LEG.dae" />
+        <mesh filename="package://f_quadruped_control/meshes/HR_UPPER_LEG.dae" />
       </geometry>
       <material name="black1" />
@@ -441,5 +441,5 @@
       <origin xyz="0 0 0" rpy="0 0 0" />
       <geometry>
-        <mesh filename="package://quadruped_description/meshes/HR_LOWER_LEG.dae" />
+        <mesh filename="package://f_quadruped_control/meshes/HR_LOWER_LEG.dae" />
       </geometry>
       <material name="black2" />
@@ -470,5 +470,5 @@
       <origin xyz="0 0 0" rpy="0 0 0" />
       <geometry>
-        <mesh filename="package://quadruped_description/meshes/HR_SHANK.dae" />
+        <mesh filename="package://f_quadruped_control/meshes/HR_SHANK.dae" />
       </geometry>
       <material name="black3" />
@@ -499,5 +499,5 @@
       <origin xyz="0 0 0" rpy="0 0 0" />
       <geometry>
-        <mesh filename="package://quadruped_description/meshes/HR_FOOT.dae" />
+        <mesh filename="package://f_quadruped_control/meshes/HR_FOOT.dae" />
       </geometry>
       <material name="red" />

Commit message: fixed lidar in sim

File: florant/f_quadruped_control/urdf/ContinuO_lidar.xacro (robot description, xacro)
@@ -3,10 +3,11 @@
   <!-- To make the robot fly -->
   <!-- Wingardium leviossssssssssssssssssa -->
-  <link name="world" />
-  <joint name="fixed_to_world" type="fixed">
-    <parent link="world" />
-    <child link="base_link" />
-    <origin xyz="0 0 0.5" rpy="0 0 0" />
-  </joint>
+  <!-- <link name="world" /> -->
+  <!---->
+  <!-- <joint name="fixed_to_world" type="fixed"> -->
+  <!--   <parent link="world" /> -->
+  <!--   <child link="base_link" /> -->
+  <!--   <origin xyz="0 0 0.5" rpy="0 0 0" /> -->
+  <!-- </joint> -->
   <!-- INCLUSIONS -->
   <xacro:include filename="$(find f_quadruped_control)/urdf/materials.xacro" />

File: florant/f_quadruped_control/urdf/sensors.xacro (robot description, xacro)
@@ -10,14 +10,18 @@
     <visual>
       <origin xyz="0 0 0" rpy="0 0 0" />
-      <geometry><cylinder radius="0.04" length="0.073" /></geometry>
+      <geometry>
+        <cylinder radius="0.04" length="0.073" />
+      </geometry>
       <material name="black" />
     </visual>
     <collision>
       <origin xyz="0 0 0" rpy="0 0 0" />
-      <geometry><cylinder radius="0.04" length="0.073" /></geometry>
+      <geometry>
+        <cylinder radius="0.04" length="0.073" />
+      </geometry>
     </collision>
   </link>
   <joint name="base_to_lidar" type="fixed">
-    <origin xyz="0.3 0 0.05" rpy="0 0.7854 0" />
+    <origin xyz="0.3 0 0.05" rpy="0 0.52 0" />
     <parent link="base" />
     <child link="os_sensor" />
@@ -26,21 +30,25 @@
   <link name="imu_link">
     <inertial>
-      <origin xyz="0 0 0" rpy="0 0 0"/>
-      <mass value="0.001"/>
-      <inertia ixx="1e-6" ixy="0" ixz="0" iyy="1e-6" iyz="0" izz="1e-6"/>
+      <origin xyz="0 0 0" rpy="0 0 0" />
+      <mass value="0.001" />
+      <inertia ixx="1e-6" ixy="0" ixz="0" iyy="1e-6" iyz="0" izz="1e-6" />
     </inertial>
     <visual>
-      <origin xyz="0 0 0" rpy="0 0 0"/>
-      <geometry><sphere radius="0.01"/></geometry>
+      <origin xyz="0 0 0" rpy="0 0 0" />
+      <geometry>
+        <sphere radius="0.01" />
+      </geometry>
     </visual>
     <collision>
-      <origin xyz="0 0 0" rpy="0 0 0"/>
-      <geometry><sphere radius="0.011"/></geometry>
+      <origin xyz="0 0 0" rpy="0 0 0" />
+      <geometry>
+        <sphere radius="0.011" />
+      </geometry>
     </collision>
   </link>
   <joint name="imu_joint" type="fixed">
-    <origin xyz="0 0 0.05" rpy="0 0 0"/>
-    <parent link="base"/>
-    <child link="imu_link"/>
+    <origin xyz="0 0 0.05" rpy="0 0 0" />
+    <parent link="base" />
+    <child link="imu_link" />
   </joint>
 </robot>
